Commit message: Add files via upload

File: ar3_description/urdf/ar3.ros2_control.xacro (robot description, xacro)
@@ -7,6 +7,10 @@
         <param name="serial_port">${serial_port}</param>
         <param name="baudrate">${baudrate}</param>
-        <!-- optional gear_ratio and limits may be read by the
-             hardware interface via <joint> entries below -->
+        <param name="gear_ratio_joint_1">10.0</param>
+        <param name="gear_ratio_joint_2">50.0</param>
+        <param name="gear_ratio_joint_3">50.0</param>
+        <param name="gear_ratio_joint_4">14.0</param>
+        <param name="gear_ratio_joint_5">1.0</param>
+        <param name="gear_ratio_joint_6">19.0</param>
       </hardware>
         <joint name="joint_1">

File: ar3_description/urdf/ar3.urdf.xacro (robot description, xacro)
@@ -24,5 +24,5 @@
   <xacro:include filename="joints/joint_6.xacro" />
   <!-- Include ros2_control configuration -->
-  <xacro:include filename="ar3.ros2_control.xacro" />
+  <!-- <xacro:include filename="ar3.ros2_control.xacro" /> -->
   <!-- Base Link -->
   <xacro:base_link />
@@ -52,6 +52,6 @@
   <xacro:link_6 />
   <!-- ros2_control configuration -->
-  <xacro:ar3_ros2_control
+  <!-- <xacro:ar3_ros2_control
     serial_port="$(arg serial_port)"
-    baudrate="$(arg baudrate)" />
+    baudrate="$(arg baudrate)" /> -->
 </robot>
